Commit message: green block, start from checkpoint

File: gym_pybullet_drones/assets/goal_position.urdf (robot description, URDF)
Before this commit: robot obstacle, 1 links, 0 joints
Links:
- link baseLink: geometry visual box size=0.2 0.2 0.02

Commit message: new reward function, green block changed

File: gym_pybullet_drones/assets/goal_position.urdf (robot description, URDF)
Before this commit: robot obstacle, 1 links, 0 joints
Links:
- link baseLink: geometry visual box size=0.25 0.25 0.25
