Commit message: env3 rew3

File: gym_pybullet_drones/assets/goal_position_sphere.urdf (robot description, URDF)
Before this commit: robot obstacle, 1 links, 0 joints
Links:
- link baseLink: geometry visual sphere radius=0.05

Commit message: new rew, bigger goal

File: gym_pybullet_drones/assets/goal_position_sphere.urdf (robot description, URDF)
Before this commit: robot obstacle, 1 links, 0 joints
Links:
- link baseLink: geometry visual sphere radius=0.15
